File: v1-cellphone.sch (EAGLE design)
At the start: 55 parts, among them J1 AVRISP, J2 ZX62D-B-5P8, U1 MCP73831, U2 MEGA1284, U3 GSM_UC15, X1 BU-SMA-V, X2 CRYSTAL, X3 CCM03-3002 R102

Commit message: Ready for review at diy devices.
Parts:
- added C10: 18pF, rcl_custom:C-EUC0603
- added C17, C18: 100nF, cellphone-rcl:C-EUC1206
- added C19, C23: 100nF 16V, cellphone-rcl:C-EUC1206
- added C20, C24: 33pF 16V, cellphone-rcl:C-EUC1206
- added C21, C25: 10pF 16V, cellphone-rcl:C-EUC1206
- added C22, C26: 100uF 16V, cellphone-rcl:C-EUC1206
- added D1, D2, D3: (no value), SparkFun-DiscreteSemi:DIODESMA
- added D4: 5.1V, SparkFun-DiscreteSemi:DIODE-ZENERSMB
- added R11: 100, v1-cellphone:CELLPHONE-RCL_R-US_R1206
- added R12: 2K, v1-cellphone:CELLPHONE-RCL_R-US_R1206
- added TP1, TP2, TP3: TPPAD1-13, testpad:TPPAD1-13
- C12, C5: value 0.1uF -> 100nF
- C14: device cellphone-rcl:C-EUC1206 -> rcl_custom:C-EUC0603
- C15: value 18pF -> 100nF
- S1: device cellphone:BUTTON-2 -> v1-cellphone:CELLPHONE_BUTTON-2
- X2: value CRYSTAL -> 16MHz
Connections:
- removed net SPK2P: U3.20-SPK2P
- removed net VCC: C11.+, C12.1, C13.1, C16.+, C4.1, J1.2-5VCC, JP3.2, JP8.2, JP9.2, LED3.A, R4.2, U1.VBAT, U2.AVCC, U2.VCC@1, U2.VCC@2, U2.VCC@3
- removed net VDD_EXT: U3.7-VDD_EXT
- removed net VUSB: C3.1, J2.VCC, LED1.A, U1.VIN
- new net 4.2V: C4.1, R11.2, U1.VBAT
- new net 4V: C11.+, C12.1, C13.1, C15.1, C16.+, C17.1, C18.1, C19.1, C20.1, C21.1, C22.1, C23.1, C24.1, C25.1, C26.1, D4.C, JP3.2, JP8.2, JP9.2, LED3.A, R11.1, R12.2, R4.2, U2.AVCC, U2.VCC@1, U2.VCC@2, U2.VCC@3, U3.50-51-VBAT_RF, U3.52-53-VBAT_BB
- new net 5V: C3.1, D1.C, D2.C, D3.C, LED1.A, U1.VIN
- new net N$10: D2.A, J1.2-5VCC
- new net N$11: D3.A, JP7.VCC
- new net N$13: TP1.TP, U3.2-AP_RDY
- new net N$14: TP2.TP, U3.7-VDD_EXT
- new net N$15: TP3.TP, U3.55-RI
- new net N$9: D1.A, J2.VCC
- net AGND: no longer U2.AREF
- net GND: now also C10.2, C17.2, C18.2, C19.2, C20.2, C21.2, C22.2, C23.2, C24.2, C25.2, C26.2, C5.1, D4.A, R12.1, U2.AREF; no longer C5.2
- net N$7: now also C10.1, X2.1; no longer C15.1, X2.2
- net N$8: now also X2.2; no longer X2.1
- net SHLD: now also C5.2; no longer C5.1
Other:
- note added: "CELLPHONE3G PROTOTYPING MODULE VERSION 0.1 7/29/2014"
- note added: "Chip Antenna"
- note added: "This board is heavily based on David Mellis' 2G Cellphone Module, with permission. It was modified by Jenner Hanni in 2014 to be 3G-capable using the Quectel UC15. It is open hardware released under the MIT License. It is a draft release and has not been built. There is no warranty. Use it at your own risk. Contact Jenner at <jeh.wicker@gmail.com> for more information"
- note removed: "?? IF USING DN,DP THEN 90 OHMS DIFF IMPEDANCE"
- note removed: "ADD THE ESD PROTECTION ESDA6V8AV6!!"
- note removed: "EITHER UNCONNECT OR ROUTE"
- note removed: "FIGURE OUT POWER"
- note removed: "REALLY, FIVE VOLTS?"
- note removed: "RI is a wakup related to UART"
- note removed: "THIS IS AN ARDUINO SERIAL PROGRAMMER"
- note removed: "TODO: - FIX GROUNDS EVERYWHERE - ALSO ADD WAY MORE BYPASS CAPS"
- note removed: "TODO: ADD A BUTTON HERE"
- note removed: "VDD_EXT PROVIDES 2.6V FOR UART LEVEL MATCH AND SIM PRESENCE DETECTION"
- note removed: "soldered antenna"
- moved on the sheet: ANT1, C1, C11, C12, C13, C15, C16, C2, C3, C4, C5, C6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

Commit message: Added notes.
Connections:
- net RESET renamed !RESET
Other:
- note added: "3G CELLPHONE MODULE"
- note added: "ATMEGA1284 MICROCONTROLLER"
- note added: "BATTERY MANAGEMENT"
- note added: "INPUT MICRO USB FOR VOLTAGE OFF BATTERY"
- note added: "PLACE ONE BYPASS CAP AT EACH VCC PIN"
- note added: "UC15 MODULE SUPPORTS BOTH 1.8V AND 3.0V SIM CARDS"
- note removed: "CHIP SUPPORTS BOTH 1.8V and 3.0V SIM CARDS"
- moved on the sheet: C1, D3, JP7, R4
Changed lines of the file:
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@@
 <text x="447.04" y="233.68" size="1.778" layer="97">Chip Antenna</text>
 <text x="449.58" y="172.72" size="1.778" layer="97">SMA or U.FL connector</text>
-<text x="447.04" y="121.92" size="1.778" layer="97">CHIP SUPPORTS BOTH 1.8V and 3.0V SIM CARDS</text>
+<text x="459.74" y="121.92" size="1.778" layer="97">UC15 MODULE SUPPORTS
+BOTH 1.8V AND 3.0V SIM CARDS</text>
 <text x="368.3" y="114.3" size="1.778" layer="94" align="center">X</text>
 <text x="472.44" y="101.6" size="1.778" layer="94" align="center">X</text>
@@
 <wire x1="513.08" y1="10.16" x2="403.86" y2="10.16" width="0.1524" layer="97"/>
 <wire x1="513.08" y1="38.1" x2="403.86" y2="38.1" width="0.1524" layer="97"/>
+<text x="63.5" y="248.92" size="1.778" layer="97">INPUT MICRO USB FOR
+VOLTAGE OFF BATTERY</text>
+<text x="160.02" y="248.92" size="1.778" layer="97">BATTERY MANAGEMENT</text>
+<text x="116.84" y="203.2" size="1.778" layer="97">PLACE ONE BYPASS CAP AT EACH VCC PIN</text>
+<text x="83.312" y="184.658" size="1.778" layer="97">ATMEGA1284
+MICROCONTROLLER</text>
+<text x="309.626" y="173.736" size="1.778" layer="97">3G CELLPHONE MODULE</text>
 </plain>
 <instances>
@@
 <instance part="R3" gate="G$1" x="406.4" y="101.6"/>
 <instance part="U2" gate="G$1" x="114.3" y="134.62"/>
-<instance part="R4" gate="G$1" x="78.74" y="193.04" rot="R90"/>
-<instance part="C1" gate="G$1" x="33.02" y="76.2"/>
+<instance part="R4" gate="G$1" x="10.16" y="195.58" rot="R90"/>
+<instance part="C1" gate="G$1" x="40.64" y="76.2"/>
 <instance part="JP3" gate="G$1" x="332.74" y="238.76" rot="MR0"/>
 <instance part="U1" gate="G$1" x="172.72" y="238.76"/>
@@
 <instance part="JP5" gate="A" x="193.04" y="93.98"/>
 <instance part="JP1" gate="A" x="180.34" y="111.76"/>
-<instance part="JP7" gate="G$1" x="20.32" y="83.82"/>
+<instance part="JP7" gate="G$1" x="27.94" y="83.82"/>
 <instance part="JP4" gate="A" x="193.04" y="134.62"/>
 <instance part="LED3" gate="G$1" x="233.68" y="236.22"/>
@@
 <instance part="J2" gate="G$1" x="71.12" y="228.6"/>
 <instance part="SUPPLY1" gate="G$1" x="223.52" y="243.84"/>
-<instance part="SUPPLY2" gate="G$1" x="78.74" y="200.66"/>
+<instance part="SUPPLY2" gate="G$1" x="10.16" y="203.2"/>
 <instance part="JP8" gate="G$1" x="332.74" y="223.52" rot="MR0"/>
 <instance part="JP9" gate="G$1" x="332.74" y="208.28" rot="MR0"/>
@@
 <instance part="R12" gate="G$1" x="210.82" y="231.14" rot="R90"/>
 <instance part="GND13" gate="1" x="210.82" y="213.36"/>
-<instance part="SUPPLY3" gate="G$1" x="38.1" y="96.52"/>
+<instance part="SUPPLY3" gate="G$1" x="45.72" y="96.52"/>
 <instance part="SUPPLY4" gate="G$1" x="22.86" y="142.24"/>
 <instance part="SUPPLY5" gate="G$1" x="104.14" y="246.38"/>
 <instance part="D1" gate="G$1" x="91.44" y="241.3"/>
 <instance part="D2" gate="G$1" x="30.48" y="137.16" rot="R180"/>
-<instance part="D3" gate="G$1" x="30.48" y="86.36"/>
+<instance part="D3" gate="G$1" x="38.1" y="86.36"/>
 <instance part="C10" gate="CE" x="43.18" y="154.94"/>
 <instance part="C14" gate="CE" x="60.96" y="154.94"/>
@@
 <segment>
 <pinref part="R4" gate="G$1" pin="2"/>
-<wire x1="78.74" y1="198.12" x2="78.74" y2="200.66" width="0.1524" layer="91"/>
+<wire x1="10.16" y1="200.66" x2="10.16" y2="203.2" width="0.1524" layer="91"/>
 <pinref part="SUPPLY2" gate="G$1" pin="4V"/>
 </segment>
@@
 <net name="GND" class="2">
 <segment>
-<wire x1="25.4" y1="91.44" x2="33.02" y2="91.44" width="0.1524" layer="91"/>
-<label x="27.94" y="91.44" size="1.778" layer="95"/>
+<wire x1="33.02" y1="91.44" x2="40.64" y2="91.44" width="0.1524" layer="91"/>
+<label x="35.56" y="91.44" size="1.778" layer="95"/>
 <pinref part="JP7" gate="G$1" pin="GND"/>
 </segment>
@@
 <net name="MIC2N" class="0">
 <segment>
-<wire x1="261.62" y1="25.4" x2="345.44" y2="25.4" width="0.1524" layer="91"/>
-<wire x1="345.44" y1="25.4" x2="345.44" y2="60.96" width="0.1524" layer="91"/>
-<label x="266.7" y="25.4" size="1.778" layer="95"/>
+<wire x1="254" y1="22.86" x2="345.44" y2="22.86" width="0.1524" layer="91"/>
+<wire x1="345.44" y1="22.86" x2="345.44" y2="60.96" width="0.1524" layer="91"/>
+<label x="266.7" y="22.86" size="1.778" layer="95"/>
 <pinref part="U3" gate="G$1" pin="26-MIC2N"/>
-<wire x1="261.62" y1="25.4" x2="261.62" y2="22.86" width="0.1524" layer="91"/>
 <pinref part="MIC1" gate="G$1" pin="2"/>
-<wire x1="261.62" y1="22.86" x2="254" y2="22.86" width="0.1524" layer="91"/>
 </segment>
 </net>
@@
 </segment>
 </net>
-<net name="RESET" class="0">
-<segment>
-<wire x1="83.82" y1="185.42" x2="78.74" y2="185.42" width="0.1524" layer="91"/>
-<wire x1="78.74" y1="185.42" x2="78.74" y2="187.96" width="0.1524" layer="91"/>
-<label x="83.82" y="185.42" size="1.778" layer="95" xref="yes"/>
+<net name="!RESET" class="0">
+<segment>
+<pinref part="C1" gate="G$1" pin="2"/>
+<wire x1="40.64" y1="71.12" x2="40.64" y2="68.58" width="0.1524" layer="91"/>
+<label x="30.48" y="68.58" size="1.778" layer="95"/>
+<wire x1="40.64" y1="68.58" x2="10.16" y2="68.58" width="0.1524" layer="91"/>
+<wire x1="10.16" y1="68.58" x2="10.16" y2="127" width="0.1524" layer="91"/>
+<pinref part="J1" gate="G$1" pin="5-RESET"/>
+<wire x1="43.18" y1="127" x2="10.16" y2="127" width="0.1524" layer="91"/>
+<label x="22.86" y="127" size="1.778" layer="95" rot="MR0"/>
+<wire x1="10.16" y1="127" x2="10.16" y2="187.96" width="0.1524" layer="91"/>
+<wire x1="60.96" y1="195.58" x2="60.96" y2="187.96" width="0.1524" layer="91"/>
+<label x="60.96" y="195.58" size="1.778" layer="95" xref="yes"/>
+<pinref part="S1" gate="G$1" pin="S"/>
+<wire x1="48.26" y1="177.8" x2="60.96" y2="177.8" width="0.1524" layer="91"/>
+<wire x1="60.96" y1="177.8" x2="60.96" y2="187.96" width="0.1524" layer="91"/>
+<pinref part="U2" gate="G$1" pin="!RESET"/>
+<wire x1="88.9" y1="177.8" x2="60.96" y2="177.8" width="0.1524" layer="91"/>
+<junction x="60.96" y="177.8"/>
+<junction x="60.96" y="187.96"/>
+<junction x="10.16" y="127"/>
 <pinref part="R4" gate="G$1" pin="1"/>
-<pinref part="S1" gate="G$1" pin="S"/>
-<wire x1="48.26" y1="177.8" x2="78.74" y2="177.8" width="0.1524" layer="91"/>
-<wire x1="78.74" y1="177.8" x2="78.74" y2="185.42" width="0.1524" layer="91"/>
-<pinref part="U2" gate="G$1" pin="!RESET"/>
-<wire x1="88.9" y1="177.8" x2="78.74" y2="177.8" width="0.1524" layer="91"/>
-<junction x="78.74" y="177.8"/>
-<junction x="78.74" y="185.42"/>
-</segment>
-<segment>
-<pinref part="C1" gate="G$1" pin="2"/>
-<wire x1="33.02" y1="71.12" x2="33.02" y2="68.58" width="0.1524" layer="91"/>
-<wire x1="33.02" y1="68.58" x2="40.64" y2="68.58" width="0.1524" layer="91"/>
-<label x="40.64" y="68.58" size="1.778" layer="95" xref="yes"/>
-</segment>
-<segment>
-<pinref part="J1" gate="G$1" pin="5-RESET"/>
-<wire x1="43.18" y1="127" x2="25.4" y2="127" width="0.1524" layer="91"/>
-<label x="25.4" y="127" size="1.778" layer="95" rot="MR0" xref="yes"/>
+<wire x1="10.16" y1="187.96" x2="60.96" y2="187.96" width="0.1524" layer="91"/>
+<wire x1="10.16" y1="187.96" x2="10.16" y2="190.5" width="0.1524" layer="91"/>
+<junction x="10.16" y="187.96"/>
 </segment>
 </net>
 <net name="N$5" class="0">
 <segment>
-<wire x1="25.4" y1="78.74" x2="33.02" y2="78.74" width="0.1524" layer="91"/>
+<wire x1="33.02" y1="78.74" x2="40.64" y2="78.74" width="0.1524" layer="91"/>
 <pinref part="C1" gate="G$1" pin="1"/>
 <pinref part="JP7" gate="G$1" pin="DTR"/>
@@
 <wire x1="88.9" y1="104.14" x2="63.5" y2="104.14" width="0.1524" layer="91"/>
 <wire x1="63.5" y1="104.14" x2="63.5" y2="83.82" width="0.1524" layer="91"/>
-<wire x1="63.5" y1="83.82" x2="25.4" y2="83.82" width="0.1524" layer="91"/>
-<label x="40.64" y="83.82" size="1.778" layer="95"/>
+<wire x1="63.5" y1="83.82" x2="33.02" y2="83.82" width="0.1524" layer="91"/>
+<label x="48.26" y="83.82" size="1.778" layer="95"/>
 <pinref part="JP7" gate="G$1" pin="TXO"/>
 </segment>
@@
 <net name="TXD0" class="0">
 <segment>
-<wire x1="66.04" y1="81.28" x2="25.4" y2="81.28" width="0.1524" layer="91"/>
-<label x="40.64" y="81.28" size="1.778" layer="95"/>
+<wire x1="66.04" y1="81.28" x2="33.02" y2="81.28" width="0.1524" layer="91"/>
+<label x="48.26" y="81.28" size="1.778" layer="95"/>
 <pinref part="JP7" gate="G$1" pin="RXI"/>
 <wire x1="66.04" y1="81.28" x2="66.04" y2="101.6" width="0.1524" layer="91"/>
@@
 <net name="5V" class="0">
 <segment>
-<wire x1="38.1" y1="86.36" x2="38.1" y2="96.52" width="0.1524" layer="91"/>
+<wire x1="45.72" y1="86.36" x2="45.72" y2="96.52" width="0.1524" layer="91"/>
 <pinref part="SUPPLY3" gate="G$1" pin="5V"/>
 <pinref part="D3" gate="G$1" pin="C"/>
-<wire x1="33.02" y1="86.36" x2="38.1" y2="86.36" width="0.1524" layer="91"/>
+<wire x1="40.64" y1="86.36" x2="45.72" y2="86.36" width="0.1524" layer="91"/>
 </segment>
 <segment>
@@
 <pinref part="JP7" gate="G$1" pin="VCC"/>
 <pinref part="D3" gate="G$1" pin="A"/>
-<wire x1="25.4" y1="86.36" x2="27.94" y2="86.36" width="0.1524" layer="91"/>
-</segment>
-</net>
+<wire x1="33.02" y1="86.36" x2="35.56" y2="86.36" width="0.1524" layer="91"/>
+</segment>
+</net>

Commit message: Version 1.2 with diode and power changes, package fixes to 0603.
Parts:
- removed D1, D2, D3: (no value), SparkFun-DiscreteSemi:DIODESMA
- removed D4: 5.1V, SparkFun-DiscreteSemi:DIODE-ZENERSMB
- removed JP1, JP5: (no value), pinhead:PINHD-1X4
- removed JP2: (no value), v1-cellphone:PINHEAD_PINHD-1X8
- removed JP3, JP8, JP9: BATTERY INPUT, SparkFun-Connectors:M02-JST-2MM-SMT
- removed JP4: (no value), pinhead:PINHD-1X3
- removed JP6: (no value), v1-cellphone:PINHEAD_PINHD-1X4
- removed JP7: (no value), cellphone:ARDUINO_SERIAL_PROGRAMSMD-NOHOLES
- removed L23: 6.8nH Murata LQG18HN6N8J00D, SmartPrj:R-EU_0603-RND
- removed L24: 3.3nH Murata LQG18HN3N3S00D, SmartPrj:R-EU_0603-RND
- removed MIC1, MIC2, SPK: (no value), pinhead:PINHD-1X2
- removed SPEAKER: SIREN, v1-cellphone:CELLPHONE_MINI-SIREN
- added C27, C28, C29, C33, C34, C35: 33pF 10V, rcl_custom:C-EU0603-B
- added C30, C31, C32, C36, C37, C38: 10pF 10V, rcl_custom:C-EU0603-B
- added J3: PA, SparkFun-Connectors:M08LOCK_LONGPADS
- added J4: PB, SparkFun-Connectors:M04LOCK_LONGPADS
- added J5: PC1, SparkFun-Connectors:M03LOCK_LONGPADS
- added J6: PC2, SparkFun-Connectors:M04LOCK_LONGPADS
- added J7: PD, SparkFun-Connectors:M04LOCK_LONGPADS
- added J8: FTDI, cellphone:ARDUINO_SERIAL_PROGRAMSMD-NOHOLES
- added J9: BATTERY INPUT, SparkFun-Connectors:M02-JST-2MM-SMT
- added L1: 6.8nH Murata LQG18HN6N8J00D, rcl_custom:L-US0603-B
- added L2: 3.3nH Murata LQG18HN3N3S00D, rcl_custom:L-US0603-B
- added LED6: VCC, adafruit:LEDCHIP-LED0603
- added Q1: MIC, adafruit:ELECTRET
- added R13: 470, rcl_custom:R-US_0603-B
- added R14: 0 ohm, rcl_custom:R-US_0603-B
- added SP1: SIREN, v1-cellphone:CELLPHONE_MINI-SIREN
- added TP4, TP5, TP6, TP7, TP8, TP9: TPPAD1-13, testpad:TPPAD1-13
- C1: value 0.1 uF -> 100nF 16V; device cellphone-rcl:C-EUC1206 -> rcl_custom:C-EU0603-B
- C10, C14: device rcl_custom:C-EUC0603 -> rcl_custom:C-EU0603-B
- C12, C15, C17, C18, C5: value 100nF -> 100nF 16V; device cellphone-rcl:C-EUC1206 -> rcl_custom:C-EU0603-B
- C13: value 100nF 50V -> 100nF 16V; device cellphone-rcl:C-EUC1206 -> rcl_custom:C-EU0603-B
- C19, C20, C21, C22, C23, C24, C25, C26, C3, C4: device cellphone-rcl:C-EUC1206 -> rcl_custom:C-EU0603-B
- C2: value 100nF 50V -> 100nF 10V; device cellphone-rcl:C-EUC1206 -> rcl_custom:C-EU0603-B
- C6, C7, C9: value 33pF -> 33pF 10V; device cellphone-rcl:C-EUC1206 -> rcl_custom:C-EU0603-B
- C8: device SmartPrj:C-EU0603-RND -> rcl_custom:C-EU0603-B
- LED1: value (none) -> 5V; device v1-cellphone:CELLPHONE-LED_LEDCHIP-LED0603 -> adafruit:LEDCHIP-LED0603
- LED2: value (none) -> 3GSTAT; device cellphone-led:LEDSMT1206 -> adafruit:LEDCHIP-LED0603
- LED3: value PWR -> VBAT; device cellphone-led:LEDSMT1206 -> adafruit:LEDCHIP-LED0603
- LED4: value 13 -> DEBUG; device cellphone-led:LEDSMT1206 -> adafruit:LEDCHIP-LED0603
- LED5: value (none) -> NETLIGHT; device cellphone-led:LEDSMT1206 -> adafruit:LEDCHIP-LED0603
- R1, R10, R2, R3, R4, R5, R6, R9: device cellphone-rcl:R-US_R1206 -> rcl_custom:R-US_0603-B
- R11, R7, R8: device v1-cellphone:CELLPHONE-RCL_R-US_R1206 -> rcl_custom:R-US_0603-B
- R12: value 2K -> 2000; device v1-cellphone:CELLPHONE-RCL_R-US_R1206 -> rcl_custom:R-US_0603-B
Connections:
- removed net 4.2V: C4.1, R11.2, U1.VBAT
- removed net 4V: C11.+, C12.1, C13.1, C15.1, C16.+, C17.1, C18.1, C19.1, C20.1, C21.1, C22.1, C23.1, C24.1, C25.1, C26.1, D4.C, JP3.2, JP8.2, JP9.2, LED3.A, R11.1, R12.2, R4.2, U2.AVCC, U2.VCC@1, U2.VCC@2, U2.VCC@3, U3.50-51-VBAT_RF, U3.52-53-VBAT_BB
- removed net ANTENA: ANT1.FEED, C8.2, L24.2, X1G$1.1
- removed net MIC1N: MIC2.2, U3.24-MIC1N
- removed net MIC1P: MIC2.1, U3.23-MIC1P
- removed net MIC2N: MIC1.2, U3.26-MIC2N
- removed net MIC2P: MIC1.1, U3.25-MIC2P
- removed net N$10: D2.A, J1.2-5VCC
- removed net N$11: D3.A, JP7.VCC
- new net ANTENNA: ANT1.FEED, C8.2, L2.2, X1G$1.1
- new net N$16: C27.2, C28.1, C30.2, C31.1, Q1.2, U3.23-MIC1P
- new net N$19: C28.2, C29.1, C31.2, C32.1, Q1.1, U3.24-MIC1N
- new net STAT: R7.1, U1.STAT
- new net VBAT: C11.+, C13.1, C16.+, C4.1, J9.2, LED3.A, R11.2, U1.VBAT
- new net VCC: C12.1, C15.1, C17.1, C18.1, C19.1, C20.1, C21.1, C22.1, C23.1, C24.1, C25.1, C26.1, LED6.A, R11.1, R12.2, R4.2, U2.AVCC, U2.VCC@1, U2.VCC@2, U2.VCC@3, U3.50-51-VBAT_RF, U3.52-53-VBAT_BB
- net 5V: now also J1.2-5VCC, J2.VCC; no longer D1.C, D2.C, D3.C
- net AGND: now also C27.1, C29.2, C30.1, C32.2, C33.1, C35.2, C36.1, C38.2, L1.1, L2.1, R14.1; no longer L23.1, L24.1
- net ANT: now also L1.2; no longer L23.2
- net GND: now also J8.GND, J9.1, R13.1, R14.2; no longer D4.A, JP3.1, JP7.GND, JP8.1, JP9.1, R7.1, U1.STAT
- net N$5: now also J8.DTR; no longer JP7.DTR
- net N$9: now also LED6.C, R13.2; no longer D1.A, J2.VCC
- net PA0: now also J3.1; no longer JP2.1
- net PA1: now also J3.2; no longer JP2.2
- net PA2: now also J3.3; no longer JP2.3
- net PA3: now also J3.4; no longer JP2.4
- net PA4: now also J3.5; no longer JP2.5
- net PA5: now also J3.6; no longer JP2.6
- net PA6: now also J3.7; no longer JP2.7
- net PA7: now also J3.8; no longer JP2.8
- net PB0: now also J4.1; no longer JP6.1
- net PB1: now also J4.2; no longer JP6.2
- net PB2: now also J4.3; no longer JP6.3
- net PB3: now also J4.4; no longer JP6.4
- net PC0: now also J5.1; no longer JP4.1
- net PC1: now also J5.2; no longer JP4.2
- net PC2: now also J5.3; no longer JP4.3
- net PC4: now also J6.1; no longer JP1.1
- net PC5: now also J6.2; no longer JP1.2
- net PC6: now also J6.3; no longer JP1.3
- net PC7: now also J6.4; no longer JP1.4
- net PD4: now also J7.1; no longer JP5.1
- net PD5: now also J7.2; no longer JP5.2
- net PD6: now also J7.3; no longer JP5.3
- net PD7: now also J7.4; no longer JP5.4
- net RXD0: now also J8.TXO; no longer JP7.TXO
- net RXD1: now also TP5.TP
- net SIM_CLKR: now also TP8.TP
- net SIM_DATA: now also TP9.TP
- net SIM_RSTR: now also TP7.TP
- net SIM_VDD: now also TP6.TP
- net SPK1N: now also C34.2, C35.1, C37.2, C38.1, SP1.1; no longer SPEAKER.1, SPK.1
- net SPK1P: now also C33.2, C34.1, C36.2, C37.1, SP1.2; no longer SPEAKER.2, SPK.2
- net TXD0: now also J8.RXI; no longer JP7.RXI
- net TXD1: now also TP4.TP
Other:
- note added: "3.7V BATTERY 3500mAh COULD BE 4.2V IF FULLY CHARGED"
- note added: "50 OHMS IMPEDANCE"
- note added: "BATTERY CHARGE MANAGEMENT CONTROLLER 500mA LIMIT"
- note added: "BATTERY CHARGER PUTS OUT 4.2V CHARGED BATTERY PUTS OUT 4.2V UC15 MAX INPUT IS 4.3V"
- note added: "CELLPHONE3G PROTOTYPING MODULE VERSION 1.2 8/2/2014"
- note added: "ELECTRET MICROPHONE"
- note added: "IF R11 IS PLACED, VOLTAGE DIVIDER CIRCUIT BRINGS LEVELS UNDER UC15 LIMIT. MAKES 3.5V FROM 3.7V AND 4V FROM 4.2V"
- note added: "PLACE R11 0 OHM AND DNP R12 FOR NO VOLT DIVIDER"
- note added: "ROUTE MIC1P AND MIC1N AS 32 OHM DIFFERENTIAL PAIR"
- note added: "ROUTE SPK1P AND SPK1N AS 32 OHM DIFFERENTIAL PAIR"
- note added: "USE THE 5V FTDI-USB CABLE COMPATIBLE WITH ARDUINO PROGRAMMING"
- note removed: "BATTERY MANAGEMENT"
- note removed: "CELLPHONE3G PROTOTYPING MODULE VERSION 0.1 7/29/2014"
- moved on the sheet: ANT1, C11, C16, J2, LED1, LED3, LED5, U1, U3, X1G2, X1G4

Commit message: Major power changes. Fixed 2.6V signal lines. Ready for review.
Parts:
- removed J6: PC2, SparkFun-Connectors:M04LOCK_LONGPADS
- removed J7: PD, SparkFun-Connectors:M04LOCK_LONGPADS
- removed LED6: VCC, adafruit:LEDCHIP-LED0603
- added C39: 2.2uF, rcl_custom:C-EU0603-B
- added Q2, Q3: NTR4501N-D, max-viz:NTR4501N-D
- added TP10, TP11, TP12, TP13, TP14, TP15, TP17: TPPAD1-13, testpad:TPPAD1-13
- added U4: TXB0104PWR, SparkFun-DigitalIC:TXB0104PWR
- C8: value 3.9pF Murata GQM1885C2A3R9BB01D -> 3.9pF 100V 0603
- J5: value PC1 -> PC; device SparkFun-Connectors:M03LOCK_LONGPADS -> SparkFun-Connectors:M08LOCK_LONGPADS
- L1: value 6.8nH Murata LQG18HN6N8J00D -> 6.8nH 430mA 0603
- L2: value 3.3nH Murata LQG18HN3N3S00D -> 3.3nH 500mA 0603
- R11: value 100 -> 4.99K
- R12: value 2000 -> 4.99K
- R13: value 470 -> 10K
Connections:
- removed net N$9: LED6.C, R13.2
- removed net PD4: J7.1, U2.(XCK1/OC1B/PCINT28)PD4
- removed net PD5: J7.2, U2.(OC1A/PCINT29)PD5
- removed net PD6: J7.3, U2.(OC2B/ICP/PCINT30)PD6
- removed net PD7: J7.4, U2.(OC2A/PCINT31)PD7
- removed net PWRKEY: U2.(TMS/PCINT19)PC3, U3.18-PWRKEY
- removed net STAT: R7.1, U1.STAT
- removed net STATUS: LED2.A, U3.54-STATUS
- removed net VCC: C12.1, C15.1, C17.1, C18.1, C19.1, C20.1, C21.1, C22.1, C23.1, C24.1, C25.1, C26.1, LED6.A, R11.1, R12.2, R4.2, U2.AVCC, U2.VCC@1, U2.VCC@2, U2.VCC@3, U3.50-51-VBAT_RF, U3.52-53-VBAT_BB
- new net !PWRKEY: Q2.D, U3.18-PWRKEY
- new net !UC15RESET: Q3.D, U3.17_!RESET
- new net 2.6V: C39.1, R13.1, TP2.TP, U3.7-VDD_EXT, U4.VCCA
- new net BATTSTATUS: R7.1, U1.STAT, U2.(OC2B/ICP/PCINT30)PD6
- new net N$10: TP10.TP, U3.11-USIM_PRESENCE
- new net N$11: TP13.TP, X3.5
- new net N$20: TP4.TP, U3.60-TXD, U4.A1
- new net N$21: TP5.TP, U3.61-RXD, U4.A2
- new net N$23: TP17.TP, U3.54-STATUS, U4.A4
- new net PC3: J5.4, U2.(TMS/PCINT19)PC3
- new net SETPWRKEY: Q2.G, R11.2, TP12.TP, U2.(XCK1/OC1B/PCINT28)PD4
- new net SETUC15RESET: Q3.G, R12.2, TP11.TP, U2.(OC1A/PCINT29)PD5
- new net UC15STATUS: LED2.A, U2.(OC2A/PCINT31)PD7, U4.B4
- net 5V: now also J8.VCC
- net GND: now also C39.2, Q2.S, Q3.S, R11.1, U4.GND; no longer R13.1
- net N$14: now also R13.2, U4.OE; no longer TP2.TP, U3.7-VDD_EXT
- net PC4: now also J5.5; no longer J6.1
- net PC5: now also J5.6; no longer J6.2
- net PC6: now also J5.7; no longer J6.3
- net PC7: now also J5.8; no longer J6.4
- net RXD1: now also TP15.TP, U4.B1; no longer TP5.TP, U3.60-TXD
- net TXD1: now also TP14.TP, U4.B2; no longer TP4.TP, U3.61-RXD
- net VBAT: now also C12.1, C15.1, C17.1, C18.1, C19.1, C20.1, C21.1, C22.1, C23.1, C24.1, C25.1, C26.1, R4.2, U2.AVCC, U2.VCC@1, U2.VCC@2, U2.VCC@3, U3.50-51-VBAT_RF, U3.52-53-VBAT_BB, U4.VCCB; no longer R11.2
Other:
- note added: "3.7V LIPO OUTPUT: COULD BE 4.2V MAX"
- note added: "ATMEGA1284 MICROCONTROLLER VBAT MAX IS 4.2V BUT IT DISCHARGES OVER TIME DO NOT ATTACH ISP, FTDI, OR USB AT THE SAME TIME."
- note added: "BATTERY CHARGER PUTS OUT 4.2V CHARGED BATTERY PUTS OUT 4.2V UC15 MAX INPUT IS 4.3V VBAT POWERS THE 3G MODULE AND THE MICROCONTROLLER"
- note added: "LEVEL TRANSLATED SIGNALS FROM 2.6V (3G) TO VBAT (MICROCONTROLLER)"
- note added: "PLACE ONE BYPASS CAP AT EACH VBAT PIN"
- note added: "PULL !PWKREY LOW TO TURN ON MODULE"
- note added: "PULL !UC15RESET LOW TO TURN ON MODULE"
- note added: "QUECTEL UC15 3G CELLPHONE MODULE"
- note added: "RESETS THE MODULE"
- note added: "SIGNAL INDICATES TO MICROCONTROLLER WHEN BATTERY IS CHARGING"
- note added: "SIGNALS TO UC15 3G MODULE"
- note added: "STATUS OF MODULE"
- note added: "TODO MAKE CELLPHONE LIBRARY OF PACKAGES LAY OUT THE BOARD MAKE BOM WRITE EVERYTHING UP REVIEW BOARD POST ON THE WEB"
- note added: "TURNS ON/OFF THE MODULE"
- note added: "VDD_EXT PROVIDES 2.6V REFERENCE OUTPUT"
- note removed: "3G CELLPHONE MODULE"
- note removed: "BATTERY CHARGER PUTS OUT 4.2V CHARGED BATTERY PUTS OUT 4.2V UC15 MAX INPUT IS 4.3V"
- note removed: "IF R11 IS PLACED, VOLTAGE DIVIDER CIRCUIT BRINGS LEVELS UNDER UC15 LIMIT. MAKES 3.5V FROM 3.7V AND 4V FROM 4.2V"
- note removed: "PLACE ONE BYPASS CAP AT EACH VCC PIN"
- note removed: "PLACE R11 0 OHM AND DNP R12 FOR NO VOLT DIVIDER"
