File: v1-cellphone.sch (EAGLE design)
At the start: 93 parts, among them J1 AVRISP, J2 ZX62D-B-5P8, J4 FTDI, J5 BATTERY INPUT, Q1 MIC, Q2 NTR4501N-D, Q3 NTR4501N-D, U1 MCP73831, U2 MEGA1284, U3 GSM_UC15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

Commit message: Final for release. Passes ERC, DRC.
Parts:
- removed C20: 33pF 16V, rcl_custom:C-EU0603-B
- removed C22: 100uF 16V, rcl_custom:C-EUC1210K
- removed JP1, JP2, JP3: (no value), SparkFun-Connectors:M04LOCK
- added J3, J6, J7: (no value), SparkFun-Connectors:M04LOCK
Connections:
- removed net PC0: U2.(SCL/PCINT16)PC0
- removed net PC1: U2.(SDA/PCINT17)PC1
- removed net PC2: U2.(TCK/PCINT18)PC2
- removed net PC3: U2.(TMS/PCINT19)PC3
- removed net PC4: U2.(TDO/PCINT20)PC4
- removed net PC5: U2.(TDI/PCINT21)PC5
- removed net PC6: U2.(TOSC1/PCINT22)PC6
- removed net PC7: U2.(TOSC2/PCINT23)PC7
- net GND: no longer C20.2, C22.2
- net PA0: now also J3.1; no longer JP1.1
- net PA1: now also J3.2; no longer JP1.2
- net PA2: now also J3.3; no longer JP1.3
- net PA3: now also J3.4; no longer JP1.4
- net PA4: now also J6.1; no longer JP2.1
- net PA5: now also J6.2; no longer JP2.2
- net PA6: now also J6.3; no longer JP2.3
- net PA7: now also J6.4; no longer JP2.4
- net PB0: now also J7.1; no longer JP3.1
- net PB1: now also J7.2; no longer JP3.2
- net PB2: now also J7.3; no longer JP3.3
- net PB3: now also J7.4; no longer JP3.4
- net VBAT: no longer C20.1, C22.1
Other:
- moved on the sheet: C19, C21
